File: test/test.kicad_pcb (KiCad board)
At the start: 2 copper layers, 1 part

Commit message: 一旦おけ
Parts:
- added D2: LED, LED_THT:LED_D3.0mm, F.Cu at (152.4, 91.4)
- moved D1 15.2 mm to (142.2, 86.4)
Changed lines of the file:
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@@
   (net 1 "unconnected-(D1-K-Pad1)")
   (net 2 "unconnected-(D1-A-Pad2)")
+  (net 3 "unconnected-(D2-K-Pad1)")
+  (net 4 "unconnected-(D2-A-Pad2)")
   (footprint "LED_THT:LED_D3.0mm" (layer "F.Cu")
-    (at 127 86.36)
+    (at 142.24 86.36)
     (descr "LED, diameter 3.0mm, 2 pins")
     (tags "LED diameter 3.0mm 2 pins")
@@
     (model "${KICAD6_3DMODEL_DIR}/LED_THT.3dshapes/LED_D3.0mm.wrl"
       (offset (xyz 0 0 0))
+      (scale (xyz 1 1 1))
+      (rotate (xyz 0 0 0))
+    )
+  )
+  (footprint "LED_THT:LED_D3.0mm" (layer "F.Cu")
+    (at 152.4 91.44)
+    (descr "LED, diameter 3.0mm, 2 pins")
+    (tags "LED diameter 3.0mm 2 pins")
+    (property "Sheetfile" "test.kicad_sch")
+    (property "Sheetname" "")
+    (property "ki_description" "Light emitting diode")
+    (property "ki_keywords" "LED diode")
+    (attr through_hole)
+    (fp_text reference "D2" (at 1.27 -2.96) (layer "F.SilkS")
+        (effects (font (size 1 1) (thickness 0.15)))
+    )
+    (fp_text value "LED" (at 1.27 2.96) (layer "F.Fab")
+        (effects (font (size 1 1) (thickness 0.15)))
+    )
+    (fp_line (start -0.29 -1.236) (end -0.29 -1.08)
+      (stroke (width 0.12) (type solid)) (layer "F.SilkS"))
+    (fp_line (start -0.29 1.08) (end -0.29 1.236)
+      (stroke (width 0.12) (type solid)) (layer "F.SilkS"))
+    (fp_arc (start -0.29 -1.235516) (mid 1.366487 -1.987659) (end 2.942335 -1.078608)
+      (stroke (width 0.12) (type solid)) (layer "F.SilkS"))
+    (fp_arc (start 0.229039 -1.08) (mid 1.270117 -1.5) (end 2.31113 -1.079837)
+      (stroke (width 0.12) (type solid)) (layer "F.SilkS"))
+    (fp_arc (start 2.31113 1.079837) (mid 1.270117 1.5) (end 0.229039 1.08)
+      (stroke (width 0.12) (type solid)) (layer "F.SilkS"))
+    (fp_arc (start 2.942335 1.078608) (mid 1.366487 1.987659) (end -0.29 1.235516)
+      (stroke (width 0.12) (type solid)) (layer "F.SilkS"))
+    (fp_line (start -1.15 -2.25) (end -1.15 2.25)
+      (stroke (width 0.05) (type solid)) (layer "F.CrtYd"))
+    (fp_line (start -1.15 2.25) (end 3.7 2.25)
+      (stroke (width 0.05) (type solid)) (layer "F.CrtYd"))
+    (fp_line (start 3.7 -2.25) (end -1.15 -2.25)
+      (stroke (width 0.05) (type solid)) (layer "F.CrtYd"))
+    (fp_line (start 3.7 2.25) (end 3.7 -2.25)
+      (stroke (width 0.05) (type solid)) (layer "F.CrtYd"))
+    (fp_line (start -0.23 -1.16619) (end -0.23 1.16619)
+      (stroke (width 0.1) (type solid)) (layer "F.Fab"))
+    (fp_arc (start -0.23 -1.16619) (mid 3.17 0.000452) (end -0.230555 1.165476)
+      (stroke (width 0.1) (type solid)) (layer "F.Fab"))
+    (fp_circle (center 1.27 0) (end 2.77 0)
+      (stroke (width 0.1) (type solid)) (fill none) (layer "F.Fab"))
+    (pad "1" thru_hole rect (at 0 0) (size 1.8 1.8) (drill 0.9) (layers "*.Cu" "*.Mask")
+      (net 3 "unconnected-(D2-K-Pad1)") (pinfunction "K") (pintype "passive"))
+    (pad "2" thru_hole circle (at 2.54 0) (size 1.8 1.8) (drill 0.9) (layers "*.Cu" "*.Mask")
+      (net 4 "unconnected-(D2-A-Pad2)") (pinfunction "A") (pintype "passive"))
+    (model "${KICAD6_3DMODEL_DIR}/LED_THT.3dshapes/LED_D3.0mm.wrl"
+      (offset (xyz 0 0 0))
