File: test/test.kicad_sch (KiCad schematic)
At the start: 1 part

Commit message: 一旦おけ
Parts:
- added D2: LED, LED_THT:LED_D3.0mm, symbol Device:LED
Other:
- moved on the sheet: D1
Changed lines of the file:
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@@
 (kicad_sch (version 20230121) (generator eeschema)
   (paper "A4")
-  (symbol (lib_id "Device:LED") (at 80.01 85.09 0) (unit 1)
+  (symbol (lib_id "Device:LED") (at 93.98 63.5 0) (unit 1)
     (in_bom yes) (on_board yes) (dnp no) (fields_autoplaced)
-    (property "Reference" "D1" (at 78.4225 78.74 0)
+    (property "Reference" "D1" (at 92.3925 57.15 0)
       (effects (font (size 1.27 1.27)))
     )
-    (property "Value" "LED" (at 78.4225 81.28 0)
+    (property "Value" "LED" (at 92.3925 59.69 0)
       (effects (font (size 1.27 1.27)))
     )
-    (property "Footprint" "LED_THT:LED_D3.0mm" (at 80.01 85.09 0)
+    (property "Footprint" "LED_THT:LED_D3.0mm" (at 93.98 63.5 0)
       (effects (font (size 1.27 1.27)) hide)
     )
-    (property "Datasheet" "~" (at 80.01 85.09 0)
+    (property "Datasheet" "~" (at 93.98 63.5 0)
       (effects (font (size 1.27 1.27)) hide)
     )
@@
         )
       )
+    )
+  )
+  (symbol (lib_id "Device:LED") (at 109.22 66.04 0) (unit 1)
+    (in_bom yes) (on_board yes) (dnp no) (fields_autoplaced)
+    (property "Reference" "D2" (at 107.6325 59.69 0)
+      (effects (font (size 1.27 1.27)))
+    )
+    (property "Value" "LED" (at 107.6325 62.23 0)
+      (effects (font (size 1.27 1.27)))
+    )
+    (property "Footprint" "LED_THT:LED_D3.0mm" (at 109.22 66.04 0)
+      (effects (font (size 1.27 1.27)) hide)
+    )
+    (property "Datasheet" "~" (at 109.22 66.04 0)
+      (effects (font (size 1.27 1.27)) hide)
+    )
+    (pin "1")
+    (pin "2")
+    (instances
+      (project "test"
+        (path "/3b301d68-3828-4d1f-a3b7-7d2f8bd3de6c"
+          (reference "D2") (unit 1)
+        )
+      )
