File: AudioAmp_v0/AudioAmp_v0.kicad_pcb (KiCad board)
At the start: 2 copper layers, 95 x 72 mm, 82 parts, among them J1 AudioJack3, J2 Conn_01x02_Pin, J3 Connector_RCJ-042, J4 Connector_RCJ-042, J5 AudioJack3, J6 Conn_01x02_Pin, J7 Conn_01x02_Pin, Q1 NMOS_ MTB7D0N6RJ3, Q2 PMOS_MTP4835I3, Q3 NMOS_BSS138, Q4 PMOS_BSS84, Q5 PMOS_BSS84, Q6 PMOS_MTP4835I3, Q7 NMOS_BSS138, Q8 NMOS_ MTB7D0N6RJ3, SW1 SW_DPDT_x2, SW2 SW_DPDT_x2, U1 MAU108, U2 NJM5532, U3 NJM5532

Commit message: ビアを増やしたり
Routing:
- net GND: track 120.9 -> 123.0 mm, vias 126 -> 312
- net Net-(U3A--): track 30.9 -> 31.8 mm

Commit message: 発注
Other:
- board text added: "JLCJLCJLCJLC"
Changed lines of the file:
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@@
     (effects (font (size 0.9 0.9) (thickness 0.11)))
+  )
+  (gr_text "JLCJLCJLCJLC" (at 46.301404 25.720308 90) (layer "F.SilkS")
+    (effects (font (size 1 1)) (justify left bottom))
   )
   (gr_text "Volume" (at 57.15 71.374 90) (layer "F.SilkS" knockout)
